File: keyboard_data/bottom_plate/bottom_plate.kicad_pcb (KiCad board)
At the start: 2 copper layers, 235 x 82.6 mm, 10 parts

Commit message: fix: adjust to prevent the screws at the four corners from interfering with the PCB
Parts:
- removed the Ref** at (44.5, 122.2)
- removed the Ref** at (274.3, 44.8)
- removed the Ref** at (274.3, 122.2)
- removed the Ref** at (44.5, 44.8)
- added Ref**: Val**, kbd_Hole:m2_Screw_Hole, F.Cu at (43.4, 43.5)
- added Ref**: Val**, kbd_Hole:m2_Screw_Hole, F.Cu at (275.8, 43.6)
- added Ref**: Val**, kbd_Hole:m2_Screw_Hole, F.Cu at (275.8, 123.1)
- added Ref**: Val**, kbd_Hole:m2_Screw_Hole, F.Cu at (43.4, 123.1)
- moved G*** 2.40 mm to (162.4, 84.9)
- moved REF** 1.10 mm to (99.7, 57.1)
- moved REF** 1.10 mm to (85.7, 43.1)
- moved REF** 1.10 mm to (99.7, 43.1)
- moved REF** 1.10 mm to (92.7, 50.1)
- moved REF** 1.10 mm to (85.7, 57.1)
Other:
- board size 235 x 82.6 mm -> 237.4 x 84.7 mm
