File: keyboard_data/assemble/rhyn-oc47-assemble.kicad_sch (KiCad schematic)
At the start: 95 parts, among them SW1 SW_PUSH, SW10 SW_PUSH, SW11 SW_PUSH, SW12 SW_PUSH, SW13 SW_PUSH, SW14 SW_PUSH, SW15 SW_PUSH, SW16 SW_PUSH, SW17 SW_PUSH, SW18 SW_PUSH, SW19 SW_PUSH, SW2 SW_PUSH, SW20 SW_PUSH, SW21 SW_PUSH, SW22 SW_PUSH, SW23 SW_PUSH, SW24 SW_PUSH, SW25 SW_PUSH, SW26 SW_PUSH, SW27 SW_PUSH, SW28 SW_PUSH, SW29 SW_PUSH, SW3 SW_PUSH, SW30 SW_PUSH, SW31 SW_PUSH, SW32 SW_PUSH, SW33 SW_PUSH, SW34 SW_PUSH, SW35 SW_PUSH, SW36 SW_PUSH, SW37 SW_PUSH, SW38 SW_PUSH, SW39 SW_PUSH, SW4 SW_PUSH, SW40 SW_PUSH, SW41 SW_PUSH, SW42 SW_PUSH, SW43 SW_PUSH, SW44 SW_PUSH, SW45 SW_PUSH, SW46 SW_PUSH, SW47 SW_PUSH, SW5 SW_PUSH, SW6 SW_PUSH, SW7 SW_PUSH, SW8 SW_PUSH, SW9 SW_PUSH, U2 RP2040-Tiny

Commit message: feat: rewire myself
Connections:
- net Col0: now also U2.9; no longer U2.0
- net Col1: now also U2.10; no longer U2.1
- net Col10: now also U2.15; no longer U2.12
- net Col11: now also U2.14; no longer U2.13
- net Col2: now also U2.11; no longer U2.4
- net Col3: now also U2.12; no longer U2.5
- net Col4: now also U2.13; no longer U2.6
- net Col5: now also U2.5; no longer U2.7
- net Col6: now also U2.6; no longer U2.8
- net Col7: now also U2.28; no longer U2.9
- net Col8: now also U2.27; no longer U2.10
- net Col9: now also U2.26; no longer U2.11
- net Row0: now also U2.0; no longer U2.14
- net Row1: now also U2.1; no longer U2.15
- net Row2: now also U2.8; no longer U2.26
- net Row3: now also U2.7; no longer U2.27
