File: keyboard_data/assemble/rhyn-oc47-assemble.kicad_pcb (KiCad board)
At the start: 2 copper layers, 228.8 x 76.2 mm, 97 parts, among them SW1 SW_PUSH, SW10 SW_PUSH, SW11 SW_PUSH, SW12 SW_PUSH, SW13 SW_PUSH, SW14 SW_PUSH, SW15 SW_PUSH, SW16 SW_PUSH, SW17 SW_PUSH, SW18 SW_PUSH, SW19 SW_PUSH, SW2 SW_PUSH, SW20 SW_PUSH, SW21 SW_PUSH, SW22 SW_PUSH, SW23 SW_PUSH, SW24 SW_PUSH, SW25 SW_PUSH, SW26 SW_PUSH, SW27 SW_PUSH, SW28 SW_PUSH, SW29 SW_PUSH, SW3 SW_PUSH, SW30 SW_PUSH, SW31 SW_PUSH, SW32 SW_PUSH, SW33 SW_PUSH, SW34 SW_PUSH, SW35 SW_PUSH, SW36 SW_PUSH, SW37 SW_PUSH, SW38 SW_PUSH, SW39 SW_PUSH, SW4 SW_PUSH, SW40 SW_PUSH, SW41 SW_PUSH, SW42 SW_PUSH, SW43 SW_PUSH, SW44 SW_PUSH, SW45 SW_PUSH, SW46 SW_PUSH, SW47 SW_PUSH, SW5 SW_PUSH, SW6 SW_PUSH, SW7 SW_PUSH, SW8 SW_PUSH, SW9 SW_PUSH, U2 RP2040-Tiny

Commit message: chore: etc
Parts:
- moved D3 16.5 mm to (84.7, 53.9), turned to -90 degrees
- moved G*** 0.91 mm to (178.6, 117.7)
- turned SW3 to 180 degrees
Routing:
- net Col2: track 158.9 -> 175.2 mm
- net Row0: track 239.5 -> 248.0 mm
- net Net-(D3-A): track 6.00 -> 5.24 mm
- net GND: vias 28 -> 50
- net (no net): vias 24 -> 0
