File: low-profile-with-trackball/pcb/low-profile-with-trackball/low-profile-with-trackball.kicad_pcb (KiCad board)
At the start: 2 copper layers, 228.8 x 76.2 mm, 138 parts, among them J2 USB_C_Receptacle_USB2.0_16P, SW1 SW_PUSH, SW10 SW_PUSH, SW11 SW_PUSH, SW12 SW_PUSH, SW13 SW_PUSH, SW14 SW_PUSH, SW15 SW_PUSH, SW16 SW_PUSH, SW17 SW_PUSH, SW18 SW_PUSH, SW19 SW_PUSH, SW2 SW_PUSH, SW20 SW_PUSH, SW21 SW_PUSH, SW22 SW_PUSH, SW23 SW_PUSH, SW24 SW_PUSH, SW25 SW_PUSH, SW26 SW_PUSH, SW27 SW_PUSH, SW28 SW_PUSH, SW29 SW_PUSH, SW3 SW_PUSH, SW30 SW_PUSH, SW31 SW_PUSH, SW32 SW_PUSH, SW33 SW_PUSH, SW34 SW_PUSH, SW35 SW_PUSH, SW36 SW_PUSH, SW37 SW_PUSH, SW38 SW_PUSH, SW39 SW_PUSH, SW4 SW_PUSH, SW40 SW_PUSH, SW41 SW_PUSH, SW42 SW_PUSH, SW43 SW_PUSH, SW44 SW_PUSH, SW45 SW_PUSH, SW46 SW_PUSH, SW47 SW_PUSH, SW48 boot, SW5 SW_PUSH, SW6 SW_PUSH, SW7 SW_PUSH, SW8 SW_PUSH, SW9 SW_PUSH, U1 RP2040, U2 W25Q16JVUXIQ, U3 PMW3610, U4 XC6206P332MR, U5 SMF05CT1G, U6 MCP1700x-180xxTT, Y1 X322512MSB4SI

Commit message: add trackball base and etc
Parts:
- removed the G*** at (189.0, 116.8)
- added G***: LOGO, LOGO, F.Cu at (112.6, 84.9)
Other:
- board text added: "rhyn47"
